Commit message: 增加部分gripper相关逻辑

File: nero/nero_ros/src/nero_description/urdf/nero_description.urdf (robot description, URDF)
Before this commit: robot nero, 13 links, 12 joints
Joints:
- joint joint1: limit lower=-2.70526 upper=0.1745329252 effort=100 velocity=5 -> lower=-2.0 upper=2.0 effort=100 velocity=5
- joint joint5: limit lower=0.001 upper=2.75 effort=100 velocity=5 -> lower=-2.0 upper=2.0 effort=100 velocity=5

File: nero/nero_ros/src/nero_description/urdf/nero_dual_arm_description.xacro (robot description, xacro)
@@ -48,4 +48,5 @@
     - joint3 左右臂均为对称全范围 [-2.75, 2.75] rad。
   -->
+  <!-- J1 upper限制到2.0；J5lower同样编导 -->
   <xacro:nero_arm
     prefix="left_"
